Commit message: meshes are a work in progress

File: nxt/trunk/nxt_description/models/sensor_array.urdf (robot description, URDF)
Before this commit: robot sensor_array, 1 links, 0 joints
Links:
- added link beam_1, mass 0.1479; collision box size=0.018 0.298 0.020; visual mesh filename=package://nxt_description/meshes/collada/beams/beam_15M.dae scale=0.001 0.001 0.001
- added link beam_2, mass 0.1479; collision box size=0.018 0.298 0.020; visual mesh filename=package://nxt_description/meshes/collada/beams/beam_15M.dae scale=0.001 0.001 0.001
- added link connector_1, mass 0.1479; collision box size=0.020 0.060 0.060; visual mesh filename=package://nxt_description/meshes/collada/connectors/beam_3M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 scale=0.001 0.001 0.001
- added link connector_2, mass 0.1479; collision box size=0.020 0.060 0.060; visual mesh filename=package://nxt_description/meshes/collada/connectors/beam_3M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 scale=0.001 0.001 0.001
- added link connector_3, mass 0.1479; collision box size=0.020 0.060 0.060; visual mesh filename=package://nxt_description/meshes/collada/connectors/beam_3M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 scale=0.001 0.001 0.001
- added link connector_4, mass 0.1479; collision box size=0.020 0.060 0.060; visual mesh filename=package://nxt_description/meshes/collada/connectors/beam_3M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 scale=0.001 0.001 0.001
- added link touch_sensor_1, mass 0.1479; collision box size=0.0595 0.0985 0.0785; visual mesh filename=package://nxt_description/meshes/collada/sensors/touch_sens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 scale=0.001 0.001 0.001
- added link ultrasonic_sensor_1, mass 0.1479; collision box size=0.1375 0.1085 0.0785; visual mesh filename=package://nxt_description/meshes/collada/sensors/ultrasonic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 scale=0.001 0.001 0.001
- link nxt_brick: geometry collision box size=0.2775 0.1795 0.100; visual mesh filename=package://nxt_description/meshes/collada/sensors/nxt_intell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 scale=0.001 0.001 0.001
Joints:
- added joint joint1: type fixed, parent world, child nxt_brick, origin xyz=0 0 0 rpy=0 0 0, axis 0 0 1
- added joint joint2: type fixed, parent nxt_brick, child beam_1, origin xyz=0.09875 0 0.090 rpy=0 1.57079 0, axis 0 0 1
- added joint joint3: type fixed, parent nxt_brick, child beam_2, origin xyz=-0.09875 0 0.090 rpy=0 1.57079 0, axis 0 0 1
- added joint joint4: type fixed, parent beam_1, child connector_1, origin xyz=0 0.120 0.020 rpy=1.57079 0 0, axis 0 1 0
- added joint joint5: type fixed, parent beam_1, child connector_2, origin xyz=0 -0.120 0.020 rpy=1.57079 0 0, axis 0 1 0
- added joint joint6: type fixed, parent beam_2, child connector_3, origin xyz=0 0.120 -0.020 rpy=1.57079 0 0, axis 0 1 0
- added joint joint7: type fixed, parent beam_2, child connector_4, origin xyz=0 -0.120 -0.020 rpy=1.57079 0 0, axis 0 1 0
- added joint joint8: type fixed, parent connector_1, child ultrasonic_sensor_1, origin xyz=0 0.020 0 rpy=1.57079 0 -1.57079, axis 1 0 0
- added joint joint9: type fixed, parent connector_2, child touch_sensor_1, origin xyz=0 0.020 0 rpy=1.57079 0 -1.57079, axis 1 0 0

Commit message: working test urdf but still need to populate the model database

File: nxt/trunk/nxt_description/models/sensor_array.urdf (robot description, URDF)
Before this commit: robot sensor_array, 9 links, 9 joints
Links:
- added link beam_3, mass 0.1479; collision box size=0.018 0.098 0.020; visual mesh filename=package://nxt_description/meshes/collada/beams/beam_5M.dae scale=0.001 0.001 0.001
- added link color_sensor_1, mass 0.1479; collision box size=0.060 0.1065 0.0785; visual mesh filename=package://nxt_description/meshes/collada/sensors/color_sens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 scale=0.001 0.001 0.001
- added link connector_5, mass 0.1479; collision box size=0.040 0.016 0.0156; visual mesh filename=package://nxt_description/meshes/collada/connectors/connect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 scale=0.001 0.001 0.001
- added link connector_6, mass 0.1479; collision box size=0.040 0.016 0.0156; visual mesh filename=package://nxt_description/meshes/collada/connectors/connect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 scale=0.001 0.001 0.001
- added link servo_1, mass 0.1479; collision box size=0.0995 0.2695 0.1115; visual mesh filename=package://nxt_description/meshes/collada/sensors/interactiv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 scale=0.001 0.001 0.001
- added link servo_1_hub, mass 0.1479; collision box size=0.030 0.058 0.058; visual mesh filename=package://nxt_description/meshes/collada/sensors/servo_hub.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 scale=0.001 0.001 0.001
Joints:
- added joint joint10: type fixed, parent connector_3, child color_sensor_1, origin xyz=0 -0.020 0 rpy=1.57079 0 -1.57079, axis 1 0 0
- added joint joint11: type fixed, parent connector_4, child servo_1, origin xyz=-0.020 -0.040 0.162 rpy=1.57079 0 1.57079, axis 1 0 0
- added joint joint12: type continuous, parent servo_1, child servo_1_hub, origin xyz=0 0 0 rpy=0 0 3.14159, axis 1 0 0
- added joint joint13: type fixed, parent servo_1_hub, child beam_3, origin xyz=0.040 0 0 rpy=0 1.57079 0, axis 1 0 0
- added joint joint14: type fixed, parent servo_1_hub, child connector_5, origin xyz=0.030 0.020 0 rpy=0 0 0, axis 1 0 0
- added joint joint15: type fixed, parent servo_1_hub, child connector_6, origin xyz=0.030 -0.020 0 rpy=0 0 0, axis 1 0 0
- joint joint9: origin xyz=0 0.020 0 rpy=1.57079 0 -1.57079 -> xyz=0 0.020 0 rpy=-1.57079 0 1.57079
