Commit message: playing with how to autogenerate the urdfs from LDR files

File: nxt/trunk/nxt_robot_2.0_kit_test/robot_model.urdf.xacro (robot description, xacro)
@@ -2,4 +2,5 @@
 <robot xmlns:xacro="http://playerstage.sourceforge.net/gazebo/xmlschema/#interface"
        name="kit_test_robot" >
+  <property name="M_PI" value="3.1415926535897931" />
   <!-- The following included files set up definitions of parts of the robot body -->
   <include filename="$(find nxt_description)/models/servos/servo_v0.urdf.xacro" />
@@ -149,5 +150,5 @@
     <parent link="nxt_brick"/>
     <child link="beam_1"/>
-    <origin xyz="0.09875 0 0.090" rpy="0 1.57079 0" />
+    <origin xyz="0.09875 0 0.090" rpy="0 ${M_PI/2} 0" />
     <axis xyz="0 0 1" />
   </joint>
@@ -155,5 +156,5 @@
     <parent link="nxt_brick"/>
     <child link="beam_2"/>
-    <origin xyz="-0.09875 0 0.090" rpy="0 1.57079 0" />
+    <origin xyz="-0.09875 0 0.090" rpy="0 ${M_PI/2} 0" />
     <axis xyz="0 0 1" />
   </joint>
@@ -161,5 +162,5 @@
     <parent link="beam_1"/>
     <child link="connector_1"/>
-    <origin xyz="0 0.120 0.020" rpy="1.57079 0 0" />
+    <origin xyz="0 0.120 0.020" rpy="${M_PI/2} 0 0" />
     <axis xyz="0 1 0" />
   </joint>
@@ -167,5 +168,5 @@
     <parent link="beam_1"/>
     <child link="connector_2"/>
-    <origin xyz="0 -0.120 0.020" rpy="1.57079 0 0" />
+    <origin xyz="0 -0.120 0.020" rpy="${M_PI/2} 0 0" />
     <axis xyz="0 1 0" />
   </joint>
@@ -173,5 +174,5 @@
     <parent link="beam_2"/>
     <child link="connector_3"/>
-    <origin xyz="0 0.120 -0.020" rpy="1.57079 0 0" />
+    <origin xyz="0 0.120 -0.020" rpy="${M_PI/2} 0 0" />
     <axis xyz="0 1 0" />
   </joint>
@@ -179,5 +180,5 @@
     <parent link="beam_2"/>
     <child link="connector_4"/>
-    <origin xyz="0 -0.120 -0.020" rpy="1.57079 0 0" />
+    <origin xyz="0 -0.120 -0.020" rpy="${M_PI/2} 0 0" />
     <axis xyz="0 1 0" />
   </joint>
@@ -185,5 +186,5 @@
     <parent link="connector_1"/>
     <child link="left_ultrasonic_link"/>
-    <origin xyz="0 0.020 0" rpy="1.57079 0 -1.57079" />
+    <origin xyz="0 0.020 0" rpy="${M_PI/2} 0 ${-M_PI/2}" />
     <axis xyz="1 0 0" />
   </joint>
@@ -191,5 +192,5 @@
     <parent link="connector_2"/>
     <child link="left_touch_link"/>
-    <origin xyz="0 0.020 0" rpy="-1.57079 0 1.57079" />
+    <origin xyz="0 0.020 0" rpy="${-M_PI/2} 0 ${M_PI/2}" />
     <axis xyz="1 0 0" />
   </joint>
@@ -197,5 +198,5 @@
     <parent link="connector_3"/>
     <child link="right_color_link"/>
-    <origin xyz="0 -0.020 0" rpy="1.57079 0 -1.57079" />
+    <origin xyz="0 -0.020 0" rpy="${M_PI/2} 0 ${-M_PI/2}" />
     <axis xyz="1 0 0" />
   </joint>
@@ -203,5 +204,5 @@
     <parent link="connector_4"/>
     <child link="right_servo_link"/>
-    <origin xyz="-0.020 -0.040 0.162" rpy="1.57079 0 1.57079" />
+    <origin xyz="-0.020 -0.040 0.162" rpy="${M_PI/2} 0 ${M_PI/2}" />
     <axis xyz="1 0 0" />
   </joint>
@@ -209,5 +210,5 @@
     <parent link="right_servo_hubs_link"/>
     <child link="beam_3"/>
-    <origin xyz="0.040 0 0" rpy="0 1.57079 0" />
+    <origin xyz="0.040 0 0" rpy="0 ${M_PI/2} 0" />
     <axis xyz="1 0 0" />
   </joint>

Commit message: working launch file for complete test robot

File: nxt/trunk/nxt_robot_2.0_kit_test/robot_model.urdf.xacro (robot description, xacro)
@@ -7,12 +7,12 @@
   <include filename="$(find nxt_description)/models/beams/beams_v0.urdf.xacro" />
   <include filename="$(find nxt_description)/models/sensors/sensors_v0.urdf.xacro" />
-  <xacro:nxt_servo_v0 name="right" reflect="1" />
+  <xacro:nxt_servo_v0 name="left" reflect="0" />
   <xacro:nxt_beams_v0 name="beam_1" length="15" />
   <xacro:nxt_beams_v0 name="beam_2" length="15" />
   <xacro:nxt_beams_v0 name="beam_3" length="5" />
   <xacro:nxt_brick_v0 name="nxt_brick" />
-  <xacro:nxt_color_v0 name="right_color_link" />
-  <xacro:nxt_touch_v0 name="left_touch_link" />
-  <xacro:nxt_ultrasonic_v0 name="left_ultrasonic_link" />
+  <xacro:nxt_color_v0 name="left_color_link" />
+  <xacro:nxt_touch_v0 name="right_touch_link" />
+  <xacro:nxt_ultrasonic_v0 name="right_ultrasonic_link" />
   <link name="connector_1">
     <inertial>
@@ -185,5 +185,5 @@
   <joint name="joint8" type="fixed">
     <parent link="connector_1"/>
-    <child link="left_ultrasonic_link"/>
+    <child link="right_ultrasonic_link"/>
     <origin xyz="0 0.020 0" rpy="${M_PI/2} 0 ${-M_PI/2}" />
     <axis xyz="1 0 0" />
@@ -191,5 +191,5 @@
   <joint name="joint9" type="fixed">
     <parent link="connector_2"/>
-    <child link="left_touch_link"/>
+    <child link="right_touch_link"/>
     <origin xyz="0 0.020 0" rpy="${-M_PI/2} 0 ${M_PI/2}" />
     <axis xyz="1 0 0" />
@@ -197,5 +197,5 @@
   <joint name="joint10" type="fixed">
     <parent link="connector_3"/>
-    <child link="right_color_link"/>
+    <child link="left_color_link"/>
     <origin xyz="0 -0.020 0" rpy="${M_PI/2} 0 ${-M_PI/2}" />
     <axis xyz="1 0 0" />
@@ -203,24 +203,24 @@
   <joint name="joint11" type="fixed">
     <parent link="connector_4"/>
-    <child link="right_servo_link"/>
+    <child link="left_servo_link"/>
     <origin xyz="-0.020 -0.040 0.162" rpy="${M_PI/2} 0 ${M_PI/2}" />
     <axis xyz="1 0 0" />
   </joint>
   <joint name="joint13" type="fixed">
-    <parent link="right_servo_hubs_link"/>
+    <parent link="left_servo_hubs_link"/>
     <child link="beam_3"/>
-    <origin xyz="0.040 0 0" rpy="0 ${M_PI/2} 0" />
+    <origin xyz="-0.040 0 0" rpy="0 ${M_PI/2} 0" />
     <axis xyz="1 0 0" />
   </joint>
   <joint name="joint14" type="fixed">
-    <parent link="right_servo_hubs_link"/>
+    <parent link="left_servo_hubs_link"/>
     <child link="connector_5"/>
-    <origin xyz="0.030 0.020 0" rpy="0 0 0" />
+    <origin xyz="-0.030 0.020 0" rpy="0 0 0" />
     <axis xyz="1 0 0" />
   </joint>
   <joint name="joint15" type="fixed">
-    <parent link="right_servo_hubs_link"/>
+    <parent link="left_servo_hubs_link"/>
     <child link="connector_6"/>
-    <origin xyz="0.030 -0.020 0" rpy="0 0 0" />
+    <origin xyz="-0.030 -0.020 0" rpy="0 0 0" />
     <axis xyz="1 0 0" />
   </joint>

Commit message: updated models for the ultrasonic sensor

File: nxt/trunk/nxt_robot_2.0_kit_test/robot_model.urdf.xacro (robot description, xacro)
@@ -186,5 +186,5 @@
     <parent link="connector_1"/>
     <child link="right_ultrasonic_link"/>
-    <origin xyz="0 0.020 0" rpy="${M_PI/2} 0 ${-M_PI/2}" />
+    <origin xyz="-0.045 0.020 -0.065" rpy="${M_PI/2} ${M_PI/2} ${-M_PI/2}" />
     <axis xyz="1 0 0" />
   </joint>
