Commit message: adding rviz display plugin

File: nxt/trunk/nxt_description/models/sensors/sensors_v0.urdf.xacro (robot description, xacro)
@@ -12,5 +12,5 @@
     <visual>
       <!-- visual origin is defined w.r.t. link local coordinate system -->
-      <origin xyz="0 0 0" rpy="0 0 0" />
+      <origin xyz="-0.065 0 -0.045" rpy="0 0 ${M_PI/2}" />
       <geometry>
         <mesh filename="package://nxt_description/meshes/collada/sensors/ultrasonic_sensor_9846.dae" scale="0.001 0.001 0.001"/>
@@ -19,5 +19,5 @@
     <collision>
       <!-- collision origin is defined w.r.t. link local coordinate system -->
-      <origin xyz="0 -0.02875 0.0305" rpy="0 0 0.0" />
+      <origin xyz="-0.065 -0.02875 -0.0155" rpy="0 0 0.0" />
       <geometry>
         <box size="0.1375 0.1085 0.0785"/>
